Commit message: Update example URDF to OSURC arm

File: urdf/T12/urdf/T12.URDF (robot description, URDF)
Before this commit: robot T12, 37 links, 36 joints
Links:
- removed link Ankle1
- removed link Ankle2
- removed link Ankle3
- removed link Ankle4
- removed link Ankle5
- removed link Ankle6
- removed link Body
- removed link Foot1
- removed link Foot2
- removed link Foot3
- removed link Foot4
- removed link Foot5
- removed link Foot6
- removed link Hip1
- removed link Hip2
- removed link Hip3
- removed link Hip4
- removed link Hip5
- removed link Hip6
- removed link Knee1
- removed link Knee2
- removed link Knee3
- removed link Knee4
- removed link Knee5
- removed link Knee6
- removed link Shin1
- removed link Shin2
- removed link Shin3
- removed link Shin4
- removed link Shin5
- removed link Shin6
- removed link Thigh1
- removed link Thigh2
- removed link Thigh3
- removed link Thigh4
- removed link Thigh5
- removed link Thigh6
- added link base_link, mass 11.8959101300667; collision mesh filename=../meshes/base_link.STL; visual mesh filename=../meshes/base_link.STL
- added link elbow, mass 11.8959101300667; collision mesh filename=../meshes/elbow.STL; visual mesh filename=../meshes/elbow.STL
- added link gripper, mass 11.8959101300667; collision mesh filename=../meshes/gripper.STL; visual mesh filename=../meshes/gripper.STL
- added link lower_arm, mass 11.8959101300667; collision mesh filename=../meshes/lower_arm.STL; visual mesh filename=../meshes/lower_arm.STL
- added link shoulder, mass 11.8959101300667; collision mesh filename=../meshes/shoulder.STL; visual mesh filename=../meshes/shoulder.STL
- added link upper_arm, mass 11.8959101300667; collision mesh filename=../meshes/upper_arm.STL; visual mesh filename=../meshes/upper_arm.STL
- added link world
- added link wrist, mass 11.8959101300667; collision mesh filename=../meshes/wrist.STL; visual mesh filename=../meshes/wrist.STL
Joints:
- removed joint AP1
- removed joint AP2
- removed joint AP3
- removed joint AP4
- removed joint AP5
- removed joint AP6
- removed joint AR1
- removed joint AR2
- removed joint AR3
- removed joint AR4
- removed joint AR5
- removed joint AR6
- removed joint HP1
- removed joint HP2
- removed joint HP3
- removed joint HP4
- removed joint HP5
- removed joint HP6
- removed joint HY1
- removed joint HY2
- removed joint HY3
- removed joint HY4
- removed joint HY5
- removed joint HY6
- removed joint KP1
- removed joint KP2
- removed joint KP3
- removed joint KP4
- removed joint KP5
- removed joint KP6
- removed joint KR1
- removed joint KR2
- removed joint KR3
- removed joint KR4
- removed joint KR5
- removed joint KR6
- added joint base_roll: type revolute, parent base_link, child shoulder, origin xyz=0.14566 -0.14314 0.11421 rpy=1.5708 0 -0.11656, axis 0 1 0, limit lower=-6.28 upper=6.28 effort=150.0 velocity=3.15
- added joint elbow_pitch: type revolute, parent upper_arm, child elbow, origin xyz=0 0 0.52362 rpy=1.4974 0 0, axis 1 0 0, limit lower=-6.28 upper=6.28 effort=150.0 velocity=3.15
- added joint elbow_roll: type revolute, parent elbow, child lower_arm, origin xyz=-0.01623 0 0.035461 rpy=0 0 0.0027091, axis 0 0 1, limit lower=-6.28 upper=6.28 effort=150.0 velocity=3.15
- added joint fixed_base: type fixed, parent world, child base_link, origin xyz=0 0 0 rpy=0 0 0
- added joint shoulder_pitch: type revolute, parent shoulder, child upper_arm, origin xyz=0.017768 0.082744 0 rpy=-1.7023 0 0, axis 1 0 0, limit lower=-6.28 upper=6.28 effort=150.0 velocity=3.15
- added joint wrist_pitch: type revolute, parent lower_arm, child wrist, origin xyz=0.052628 0 0.35621 rpy=-0.11133 0 3.1416, axis 1 0 0, limit lower=-6.28 upper=6.28 effort=150.0 velocity=3.15
- added joint wrist_roll: type revolute, parent wrist, child gripper, origin xyz=-0.069133 0 0.053575 rpy=1.5708 0 -2.9823, axis 0 1 0, limit lower=-6.28 upper=6.28 effort=150.0 velocity=3.15

File: urdf/T12/urdf/T12_flipped.URDF (robot description, URDF)
Before this commit: robot T12, 37 links, 36 joints
Links:
- removed link Ankle1
- removed link Ankle2
- removed link Ankle3
- removed link Ankle4
- removed link Ankle5
- removed link Ankle6
- removed link Body
- removed link Foot1
- removed link Foot2
- removed link Foot3
- removed link Foot4
- removed link Foot5
- removed link Foot6
- removed link Hip1
- removed link Hip2
- removed link Hip3
- removed link Hip4
- removed link Hip5
- removed link Hip6
- removed link Knee1
- removed link Knee2
- removed link Knee3
- removed link Knee4
- removed link Knee5
- removed link Knee6
- removed link Shin1
- removed link Shin2
- removed link Shin3
- removed link Shin4
- removed link Shin5
- removed link Shin6
- removed link Thigh1
- removed link Thigh2
- removed link Thigh3
- removed link Thigh4
- removed link Thigh5
- removed link Thigh6
- added link base_link, mass 11.8959101300667; collision mesh filename=../meshes/base_link.STL; visual mesh filename=../meshes/base_link.STL
- added link elbow, mass 11.8959101300667; collision mesh filename=../meshes/elbow.STL; visual mesh filename=../meshes/elbow.STL
- added link gripper, mass 11.8959101300667; collision mesh filename=../meshes/gripper.STL; visual mesh filename=../meshes/gripper.STL
- added link lower_arm, mass 11.8959101300667; collision mesh filename=../meshes/lower_arm.STL; visual mesh filename=../meshes/lower_arm.STL
- added link shoulder, mass 11.8959101300667; collision mesh filename=../meshes/shoulder.STL; visual mesh filename=../meshes/shoulder.STL
- added link upper_arm, mass 11.8959101300667; collision mesh filename=../meshes/upper_arm.STL; visual mesh filename=../meshes/upper_arm.STL
- added link world
- added link wrist, mass 11.8959101300667; collision mesh filename=../meshes/wrist.STL; visual mesh filename=../meshes/wrist.STL
Joints:
- removed joint AP1
- removed joint AP2
- removed joint AP3
- removed joint AP4
- removed joint AP5
- removed joint AP6
- removed joint AR1
- removed joint AR2
- removed joint AR3
- removed joint AR4
- removed joint AR5
- removed joint AR6
- removed joint HP1
- removed joint HP2
- removed joint HP3
- removed joint HP4
- removed joint HP5
- removed joint HP6
- removed joint HY1
- removed joint HY2
- removed joint HY3
- removed joint HY4
- removed joint HY5
- removed joint HY6
- removed joint KP1
- removed joint KP2
- removed joint KP3
- removed joint KP4
- removed joint KP5
- removed joint KP6
- removed joint KR1
- removed joint KR2
- removed joint KR3
- removed joint KR4
- removed joint KR5
- removed joint KR6
- added joint base_roll: type revolute, parent base_link, child shoulder, origin xyz=0.14566 -0.14314 0.11421 rpy=1.5708 0 -0.11656, axis 0 1 0, limit lower=-6.28 upper=6.28 effort=150.0 velocity=3.15
- added joint elbow_pitch: type revolute, parent upper_arm, child elbow, origin xyz=0 0 0.52362 rpy=1.4974 0 0, axis 1 0 0, limit lower=-6.28 upper=6.28 effort=150.0 velocity=3.15
- added joint elbow_roll: type revolute, parent elbow, child lower_arm, origin xyz=-0.01623 0 0.035461 rpy=0 0 0.0027091, axis 0 0 1, limit lower=-6.28 upper=6.28 effort=150.0 velocity=3.15
- added joint fixed_base: type fixed, parent world, child base_link, origin xyz=0 0 0 rpy=0 0 0
- added joint shoulder_pitch: type revolute, parent shoulder, child upper_arm, origin xyz=0.017768 0.082744 0 rpy=-1.7023 0 0, axis 1 0 0, limit lower=-6.28 upper=6.28 effort=150.0 velocity=3.15
- added joint wrist_pitch: type revolute, parent lower_arm, child wrist, origin xyz=0.052628 0 0.35621 rpy=-0.11133 0 3.1416, axis 1 0 0, limit lower=-6.28 upper=6.28 effort=150.0 velocity=3.15
- added joint wrist_roll: type revolute, parent wrist, child gripper, origin xyz=-0.069133 0 0.053575 rpy=1.5708 0 -2.9823, axis 0 1 0, limit lower=-6.28 upper=6.28 effort=150.0 velocity=3.15

File: urdf/T12/urdf/T12_wrong_axes.orig.URDF (robot description, URDF)
Before this commit: robot T12, 37 links, 36 joints
Links:
- removed link Ankle1
- removed link Ankle2
- removed link Ankle3
- removed link Ankle4
- removed link Ankle5
- removed link Ankle6
- removed link Body
- removed link Foot1
- removed link Foot2
- removed link Foot3
- removed link Foot4
- removed link Foot5
- removed link Foot6
- removed link Hip1
- removed link Hip2
- removed link Hip3
- removed link Hip4
- removed link Hip5
- removed link Hip6
- removed link Knee1
- removed link Knee2
- removed link Knee3
- removed link Knee4
- removed link Knee5
- removed link Knee6
- removed link Shin1
- removed link Shin2
- removed link Shin3
- removed link Shin4
- removed link Shin5
- removed link Shin6
- removed link Thigh1
- removed link Thigh2
- removed link Thigh3
- removed link Thigh4
- removed link Thigh5
- removed link Thigh6
- added link base_link, mass 11.8959101300667; collision mesh filename=../meshes/base_link.STL; visual mesh filename=../meshes/base_link.STL
- added link elbow, mass 11.8959101300667; collision mesh filename=../meshes/elbow.STL; visual mesh filename=../meshes/elbow.STL
- added link gripper, mass 11.8959101300667; collision mesh filename=../meshes/gripper.STL; visual mesh filename=../meshes/gripper.STL
- added link lower_arm, mass 11.8959101300667; collision mesh filename=../meshes/lower_arm.STL; visual mesh filename=../meshes/lower_arm.STL
- added link shoulder, mass 11.8959101300667; collision mesh filename=../meshes/shoulder.STL; visual mesh filename=../meshes/shoulder.STL
- added link upper_arm, mass 11.8959101300667; collision mesh filename=../meshes/upper_arm.STL; visual mesh filename=../meshes/upper_arm.STL
- added link world
- added link wrist, mass 11.8959101300667; collision mesh filename=../meshes/wrist.STL; visual mesh filename=../meshes/wrist.STL
Joints:
- removed joint AP1
- removed joint AP2
- removed joint AP3
- removed joint AP4
- removed joint AP5
- removed joint AP6
- removed joint AR1
- removed joint AR2
- removed joint AR3
- removed joint AR4
- removed joint AR5
- removed joint AR6
- removed joint HP1
- removed joint HP2
- removed joint HP3
- removed joint HP4
- removed joint HP5
- removed joint HP6
- removed joint HY1
- removed joint HY2
- removed joint HY3
- removed joint HY4
- removed joint HY5
- removed joint HY6
- removed joint KP1
- removed joint KP2
- removed joint KP3
- removed joint KP4
- removed joint KP5
- removed joint KP6
- removed joint KR1
- removed joint KR2
- removed joint KR3
- removed joint KR4
- removed joint KR5
- removed joint KR6
- added joint base_roll: type revolute, parent base_link, child shoulder, origin xyz=0.14566 -0.14314 0.11421 rpy=1.5708 0 -0.11656, axis 0 1 0, limit lower=-6.28 upper=6.28 effort=150.0 velocity=3.15
- added joint elbow_pitch: type revolute, parent upper_arm, child elbow, origin xyz=0 0 0.52362 rpy=1.4974 0 0, axis 1 0 0, limit lower=-6.28 upper=6.28 effort=150.0 velocity=3.15
- added joint elbow_roll: type revolute, parent elbow, child lower_arm, origin xyz=-0.01623 0 0.035461 rpy=0 0 0.0027091, axis 0 0 1, limit lower=-6.28 upper=6.28 effort=150.0 velocity=3.15
- added joint fixed_base: type fixed, parent world, child base_link, origin xyz=0 0 0 rpy=0 0 0
- added joint shoulder_pitch: type revolute, parent shoulder, child upper_arm, origin xyz=0.017768 0.082744 0 rpy=-1.7023 0 0, axis 1 0 0, limit lower=-6.28 upper=6.28 effort=150.0 velocity=3.15
- added joint wrist_pitch: type revolute, parent lower_arm, child wrist, origin xyz=0.052628 0 0.35621 rpy=-0.11133 0 3.1416, axis 1 0 0, limit lower=-6.28 upper=6.28 effort=150.0 velocity=3.15
- added joint wrist_roll: type revolute, parent wrist, child gripper, origin xyz=-0.069133 0 0.053575 rpy=1.5708 0 -2.9823, axis 0 1 0, limit lower=-6.28 upper=6.28 effort=150.0 velocity=3.15
